Commit message: Change os1 bag links to os bag links. i.e. os1_imu to os_imu

File: cartographer_ros/urdf/os1_sensor.urdf (robot description, URDF)
Before this commit: robot os1_sensor, 5 links, 4 joints
Links:
- removed link os1_imu
- removed link os1_lidar
- added link os_imu; visual box size=0.06 0.04 0.02
- added link os_lidar; visual cylinder length=0.07 radius=0.05
Joints:
- joint imu_link_joint: child os1_imu -> os_imu
- joint os1_link_joint: child os1_lidar -> os_lidar

File: ouster_description/urdf/OS1-128.urdf.xacro (robot description, xacro)
@@ -2,5 +2,5 @@
 <robot xmlns:xacro="http://www.ros.org/wiki/xacro" name="OS1-128">
   <xacro:property name="M_PI" value="3.1415926535897931" />
-  <xacro:macro name="OS1-128" params="*origin parent:=base_link name:=os1_sensor topic_points:=/os_cloud_node/points topic_imu:=/os_cloud_node/imu hz:=10 lasers:=128 samples:=2048 min_range:=0.9 max_range:=75.0 noise:=0.008 min_angle:=-${M_PI} max_angle:=${M_PI} lidar_link:=os1_lidar imu_link:=os1_imu vfov_min:=-.26 vfov_max:=.26">
+  <xacro:macro name="OS1-128" params="*origin parent:=base_link name:=os1_sensor topic_points:=/os_cloud_node/points topic_imu:=/os_cloud_node/imu hz:=10 lasers:=128 samples:=2048 min_range:=0.9 max_range:=75.0 noise:=0.008 min_angle:=-${M_PI} max_angle:=${M_PI} lidar_link:=os_lidar imu_link:=os_imu vfov_min:=-.26 vfov_max:=.26">
     <joint name="${name}_mount_joint" type="fixed">
       <xacro:insert_block name="origin" />
