Commit message: Change os1 to os throughout to be product line agnostic

File: cartographer_ros/urdf/os_sensor.urdf (robot description, URDF)
Before this commit: robot os1_sensor, 5 links, 4 joints
Links:
- removed link os1
- removed link os1_sensor
- added link os
- added link os_sensor
Joints:
- joint imu_link_joint: parent os1_sensor -> os_sensor
- joint os1_link_joint: parent os1_sensor -> os_sensor
- joint os1_link_joint_legacy: child os1 -> os
- joint sensor_link_joint: child os1_sensor -> os_sensor

File: ouster_description/urdf/OS-128.urdf.xacro (robot description, xacro)
@@ -1,6 +1,6 @@
 <?xml version="1.0"?>
-<robot xmlns:xacro="http://www.ros.org/wiki/xacro" name="OS1-128">
+<robot xmlns:xacro="http://www.ros.org/wiki/xacro" name="OS-128">
   <xacro:property name="M_PI" value="3.1415926535897931" />
-  <xacro:macro name="OS1-128" params="*origin parent:=base_link name:=os1_sensor topic_points:=/os_cloud_node/points topic_imu:=/os_cloud_node/imu hz:=10 lasers:=128 samples:=2048 min_range:=0.9 max_range:=75.0 noise:=0.008 min_angle:=-${M_PI} max_angle:=${M_PI} lidar_link:=os_lidar imu_link:=os_imu vfov_min:=-.26 vfov_max:=.26">
+  <xacro:macro name="OS-128" params="*origin parent:=base_link name:=os_sensor topic_points:=/os_cloud_node/points topic_imu:=/os_cloud_node/imu hz:=10 lasers:=128 samples:=2048 min_range:=0.9 max_range:=75.0 noise:=0.008 min_angle:=-${M_PI} max_angle:=${M_PI} lidar_link:=os_lidar imu_link:=os_imu vfov_min:=-.26 vfov_max:=.26">
     <joint name="${name}_mount_joint" type="fixed">
       <xacro:insert_block name="origin" />
@@ -24,5 +24,5 @@
          <origin xyz="0 0 0.0" rpy="0 0 1.5707" />
          <geometry>
-	         <mesh filename="package://ouster_description/meshes/os1_128.dae" />
+	         <mesh filename="package://ouster_description/meshes/os_128.dae" />
            <!-- <cylinder length="0.073" radius="0.04" /> -->
          </geometry>
@@ -45,5 +45,5 @@
     <!-- Gazebo requires the ouster_gazebo_plugins package -->
     <gazebo reference="${name}">
-        <sensor type="ray" name="${name}-OS1-128">
+        <sensor type="ray" name="${name}-OS-128">
           <pose>0 0 0 0 0 0</pose>
           <visualize>false</visualize>

File: ouster_description/urdf/example.urdf.xacro (robot description, xacro)
@@ -1,4 +1,4 @@
 <?xml version="1.0"?>
-<robot xmlns:xacro="http://www.ros.org/wiki/xacro" name="os1_example">
+<robot xmlns:xacro="http://www.ros.org/wiki/xacro" name="os_example">
   <!-- Base Footprint -->
   <link name="base_footprint" />
@@ -28,7 +28,7 @@
     </inertial>
   </link>
-  <xacro:include filename="$(find ouster_description)/urdf/OS1-64.urdf.xacro"/>
-  <OS1-64 parent="base_link" name="os1_sensor" hz="10" samples="220">
+  <xacro:include filename="$(find ouster_description)/urdf/OS-128.urdf.xacro"/>
+  <OS-128 parent="base_link" name="os_sensor" hz="10" samples="220">
     <origin xyz="0 0 1.2" rpy="0 0 0" />
-  </OS1-64>
+  </OS-128>
 </robot>
